Commit message: 优化 调试

File: src/arm_description/urdf/panther_description.urdf (robot description, URDF)
Before this commit: robot panther_description, 10 links, 9 joints
Joints:
- joint gripper_1_joint: axis 0 0 1 -> (none); limit lower=-0.06 upper=0.06 effort=0.18 velocity=1 -> (none); type prismatic -> fixed
- joint gripper_2_joint: axis 0 0 1 -> (none); limit lower=-0.06 upper=0.06 effort=0.18 velocity=1 -> (none); mimic joint=gripper_1_joint multiplier=-1 offset=0 -> (none); type prismatic -> fixed

File: src/arm_description/urdf/panther_gazebo_control.xacro (robot description, xacro)
@@ -24,5 +24,5 @@
             <command_interface name="effort"/>
             <state_interface name="position">
-                <param name="initial_value">-0.785</param>
+                <param name="initial_value">-0.5</param>
             </state_interface>
             <state_interface name="velocity"/>
@@ -32,5 +32,5 @@
             <command_interface name="effort"/>
             <state_interface name="position">
-                <param name="initial_value">1.57</param>
+                <param name="initial_value">0.5</param>
             </state_interface>
             <state_interface name="velocity"/>
@@ -61,5 +61,7 @@
             <state_interface name="effort"/>
         </joint>
-        <!-- Gripper joint -->
+        <!-- Gripper joints - 现在是固定关节，不需要控制接口 -->
+        <!-- 如果需要恢复夹爪控制，取消下面的注释并在URDF中改回prismatic -->
+        <!--
         <joint name="gripper_1_joint">
             <command_interface name="effort"/>
@@ -68,15 +70,18 @@
             <state_interface name="effort"/>
         </joint>
+        <joint name="gripper_2_joint">
+            <command_interface name="effort"/>
+            <state_interface name="position"/>
+            <state_interface name="velocity"/>
+            <state_interface name="effort"/>
+        </joint>
+        -->
     </ros2_control>
     <!-- Gazebo ROS2 Control 插件配置 -->
     <gazebo>
         <plugin filename="libgazebo_ros2_control.so" name="gazebo_ros2_control">
-            <!-- 指定控制器配置文件 -->
+            <robot_param>robot_description</robot_param>
+            <robot_param_node>robot_state_publisher</robot_param_node>
             <parameters>$(find arm_rl_sim)/config/robot_control.yaml</parameters>
-            <!-- 自动激活控制器（关键！） -->
-            <controller_manager_name>controller_manager</controller_manager_name>
-            <ros>
-                <namespace>/</namespace>
-            </ros>
         </plugin>
     </gazebo>
